Commit message: 7.10 增大速度/偏向速度方向探索

File: src/unitree_guide/unitree_ros/robots/a1_description/xacro/gazebo.xacro (robot description, xacro)
@@ -319,5 +319,6 @@
     </gazebo>
      <!-- gazebo livox mid360 plugins -->
-    <xacro:property name="M_PI" value="3.14159"/>
+    <!--下采样次数，初始值为1，射线ray 数量约等于 samples / downsample-->
+    <!-- <xacro:property name="M_PI" value="3.14159"/>
     <gazebo reference="laser_livox">
         <sensor type="ray" name="laser_livox">
@@ -354,5 +355,5 @@
             <visualize>false</visualize>
                     <samples>24000</samples>
-                    <downsample>3</downsample>  <!--下采样次数，初始值为1，射线ray 数量约等于 samples / downsample-->
+                    <downsample>3</downsample>
                     <csv_file_name>$(find a1_description)/scan_mode/mid360.csv</csv_file_name>
                     <ros_topic>/scan</ros_topic>
@@ -360,5 +361,5 @@
             </plugin>
         </sensor>
-    </gazebo>
+    </gazebo> -->
     <!-- gazebo livox imu-link plugins -->
     <gazebo reference="livox_imu_link">
