Commit message: 7.13加入视觉测试插件

File: src/unitree_guide/unitree_ros/robots/a1_description/xacro/robot.xacro (robot description, xacro)
@@ -2,4 +2,18 @@
 <robot name="a1" xmlns:xacro="http://www.ros.org/wiki/xacro">
     <xacro:arg name="DEBUG" default="false"/>
+    <xacro:arg name="ENABLE_REALSENSE" default="true"/>
+    <xacro:arg name="ENABLE_LIVOX" default="true"/>
+    <xacro:arg name="ENABLE_CAMERA" default="true"/>
+    <xacro:arg name="CONTACT_UPDATE_RATE" default="100"/>
+    <xacro:arg name="IMU_UPDATE_RATE" default="1000"/>
+    <xacro:arg name="LIVOX_UPDATE_RATE" default="10"/>
+    <xacro:arg name="LIVOX_SAMPLES" default="24000"/>
+    <xacro:arg name="LIVOX_DOWNSAMPLE" default="1"/>
+    <xacro:arg name="CAMERA_UPDATE_RATE" default="30"/>
+    <xacro:arg name="CAMERA_WIDTH" default="800"/>
+    <xacro:arg name="CAMERA_HEIGHT" default="800"/>
+    <xacro:arg name="REALSENSE_UPDATE_RATE" default="10"/>
+    <xacro:arg name="REALSENSE_WIDTH" default="640"/>
+    <xacro:arg name="REALSENSE_HEIGHT" default="480"/>
     <xacro:include filename="$(find a1_description)/xacro/const.xacro"/>
     <xacro:include filename="$(find a1_description)/xacro/materials.xacro"/>
@@ -214,4 +228,23 @@
         xyz="0 0 1" />
     </joint>
+    <link name="front_camera">
+        <inertial>
+            <mass value="0.001"/>
+            <origin rpy="0 0 0" xyz="0 0 0"/>
+            <inertia ixx="0.0001" ixy="0" ixz="0" iyy="0.0001" iyz="0" izz="0.0001"/>
+        </inertial>
+        <visual>
+            <origin rpy="0 0 0" xyz="0 0 0"/>
+            <geometry>
+                <box size="0.03 0.04 0.025"/>
+            </geometry>
+            <material name="black"/>
+        </visual>
+    </link>
+    <joint name="front_camera_joint" type="fixed">
+        <parent link="base"/>
+        <child link="front_camera"/>
+        <origin xyz="0.32 0 0.10" rpy="0 0 0"/>
+    </joint>
     <xacro:leg name="FR" mirror="-1" mirror_dae="False" front_hind="1" front_hind_dae="True">
         <origin rpy="0 0 0" xyz="${leg_offset_x} ${-leg_offset_y} 0"/>
